Commit message: Complete Digital Twin

File: arduino_bot_ws/src/arduino_bot_description/urdf/arduinobot.urdf.xacro (robot description, xacro)
@@ -21,4 +21,45 @@
         </visual>
     </link>
+    <link name="forward_drive_arm">
+        <visual>
+            <origin rpy="0 -${PI/2} ${PI/2}" xyz="0.19 0.06 -0.08" />
+            <geometry>
+                <mesh filename="package://arduino_bot_description/mesh/forward_drive_arm.STL" scale="0.01 0.01 0.01" />
+            </geometry>
+        </visual>
+    </link>
+    <link name="horizontal_arm">
+        <visual>
+            <origin rpy="${PI/2} 0 ${PI/2}" xyz="-0.03 -0.4 -0.06" />
+            <geometry>
+                <mesh filename="package://arduino_bot_description/mesh/horizontal_arm.STL" scale="0.01 0.01 0.01" />
+            </geometry>
+        </visual>
+    </link>
+    <link name="claw_support">
+        <visual>
+            <origin rpy="0 0 ${PI/2}" xyz="0 -0.05 -0.15" />
+            <geometry>
+                <mesh filename="package://arduino_bot_description/mesh/claw_support.STL" scale="0.01 0.01 0.01" />
+            </geometry>
+        </visual>
+    </link>
+    <link name="gripper_right">
+        <visual>
+            <origin rpy="0 0 -${PI/2}" xyz="-0.1 0.5 -0.1" />
+            <geometry>
+                <mesh filename="package://arduino_bot_description/mesh/right_finger.STL" scale="0.01 0.01 0.01" />
+            </geometry>
+        </visual>
+    </link>
+    <link name="gripper_left">
+        <visual>
+            <origin rpy="0 0 -${PI/2}" xyz="-0.04 0.5 -0.1" />
+            <geometry>
+                <mesh filename="package://arduino_bot_description/mesh/left_finger.STL" scale="0.01 0.01 0.01" />
+            </geometry>
+        </visual>
+    </link>
+    <link name="tool_link" />
     <joint name="virtual_joint" type="fixed">
         <parent link="world"/>
@@ -33,3 +74,42 @@
         <limit lower="-${PI/2}" upper="${PI/2}" effort="${effort}" velocity="${velocity}" />
     </joint>
+    <joint name="joint_2" type="revolute">
+        <parent link="base_plate"/>
+        <child link="forward_drive_arm"/>
+        <origin rpy="0 0 0" xyz="-0.02 0 0.350" />
+        <axis xyz="1 0 0" />
+        <limit lower="-${PI/2}" upper="${PI/2}" effort="${effort}" velocity="${velocity}" />
+    </joint>
+    <joint name="joint_3" type="revolute">
+        <parent link="forward_drive_arm"/>
+        <child link="horizontal_arm"/>
+        <origin rpy="0 0 0" xyz="0 0 0.8" />
+        <axis xyz="1 0 0" />
+        <limit lower="-${PI/2}" upper="${PI/2}" effort="${effort}" velocity="${velocity}" />
+    </joint>
+    <joint name="horizontal_arm_to_claw_support" type="fixed">
+        <parent link="horizontal_arm"/>
+        <child link="claw_support"/>
+        <origin rpy="0 0 0" xyz="0 0.82 0" />
+    </joint>
+    <joint name="joint_4" type="revolute">
+        <parent link="claw_support"/>
+        <child link="gripper_right"/>
+        <origin rpy="0 0 0" xyz="-0.04 0.13 -0.1" />
+        <axis xyz="0 0 1" />
+        <limit lower="-${PI/2}" upper="0" effort="${effort}" velocity="${velocity}" />
+    </joint>
+    <joint name="joint_5" type="revolute">
+        <parent link="claw_support"/>
+        <child link="gripper_left"/>
+        <origin rpy="0 0 0" xyz="-0.2 0.13 -0.1" />
+        <axis xyz="0 0 1" />
+        <limit lower="0" upper="${PI/2}" effort="${effort}" velocity="${velocity}" />
+        <mimic joint="joint_4" offset="0" multiplier="-1" />
+    </joint>
+    <joint name="gripper_right" type="fixed">
+        <parent link="gripper_right"/>
+        <child link="tool_link"/>
+        <origin rpy="0 0 0" xyz="0 0 0" />
+    </joint>
 </robot>

Commit message: Python ROS Services : Client&Server

File: arduino_bot_ws/src/arduino_bot_description/urdf/arduinobot.urdf.xacro (robot description, xacro)
@@ -4,6 +4,25 @@
     <xacro:property name="effort" value="30" />>
     <xacro:property name="velocity" value="10" />>
+    <xacro:macro name="default_inertial" params="mass">
+        <inertial>
+            <mass value="${mass}" />
+            <inertia ixx="1" ixy="0" ixz="0" iyy="1" iyz="0" izz="1" />
+        </inertial>
+    </xacro:macro>
+    <xacro:macro name="default_transmission" params="number">
+        <transmission name="transmission_${number}">
+            <type>transmission_interface/SimpleTransmission</type>
+            <joint name="joint_${number}">
+                <hardwareInterface>hardware_interface/PositionJointInterface</hardwareInterface>
+            </joint>
+            <actuator name="motor_${number}">
+                <hardwareInterface>hardware_interface/PositionJointInterface</hardwareInterface>
+                <mechanicalReduction>1</mechanicalReduction>
+            </actuator>
+        </transmission>
+    </xacro:macro>
     <link name="world" />
     <link name="base_link">
+        <xacro:default_inertial mass="1.0" />
         <visual>
             <origin rpy="0 0 0" xyz="-0.5 -0.5 0" />
@@ -12,6 +31,13 @@
             </geometry>
         </visual>
+        <collision>
+            <origin rpy="0 0 0" xyz="-0.5 -0.5 0" />
+            <geometry>
+                <mesh filename="package://arduino_bot_description/mesh/basement.STL" scale="0.01 0.01 0.01" />
+            </geometry>
+        </collision>
     </link>
     <link name="base_plate">
+        <xacro:default_inertial mass="0.1" />
         <visual>
             <origin rpy="0 0 0" xyz="-0.39 -0.39 -0.56" />
@@ -20,6 +46,13 @@
             </geometry>
         </visual>
+        <collision>
+            <origin rpy="0 0 0" xyz="-0.39 -0.39 -0.56" />
+            <geometry>
+                <mesh filename="package://arduino_bot_description/mesh/base_plate.STL" scale="0.01 0.01 0.01" />
+            </geometry>
+        </collision>>
     </link>
     <link name="forward_drive_arm">
+        <xacro:default_inertial mass="0.1" />
         <visual>
             <origin rpy="0 -${PI/2} ${PI/2}" xyz="0.19 0.06 -0.08" />
@@ -28,6 +61,13 @@
             </geometry>
         </visual>
+        <collision>
+            <origin rpy="0 -${PI/2} ${PI/2}" xyz="0.19 0.06 -0.08" />
+            <geometry>
+                <mesh filename="package://arduino_bot_description/mesh/forward_drive_arm.STL" scale="0.01 0.01 0.01" />
+            </geometry>
+        </collision>
     </link>
     <link name="horizontal_arm">
+        <xacro:default_inertial mass="0.1" />
         <visual>
             <origin rpy="${PI/2} 0 ${PI/2}" xyz="-0.03 -0.4 -0.06" />
@@ -36,6 +76,13 @@
             </geometry>
         </visual>
+        <collision>
+            <origin rpy="${PI/2} 0 ${PI/2}" xyz="-0.03 -0.4 -0.06" />
+            <geometry>
+                <mesh filename="package://arduino_bot_description/mesh/horizontal_arm.STL" scale="0.01 0.01 0.01" />
+            </geometry>
+        </collision>
     </link>
     <link name="claw_support">
+        <xacro:default_inertial mass="0.05" />
         <visual>
             <origin rpy="0 0 ${PI/2}" xyz="0 -0.05 -0.15" />
@@ -44,6 +91,13 @@
             </geometry>
         </visual>
+        <collision>
+            <origin rpy="0 0 ${PI/2}" xyz="0 -0.05 -0.15" />
+            <geometry>
+                <mesh filename="package://arduino_bot_description/mesh/claw_support.STL" scale="0.01 0.01 0.01" />
+            </geometry>
+        </collision>
     </link>
     <link name="gripper_right">
+        <xacro:default_inertial mass="0.01" />
         <visual>
             <origin rpy="0 0 -${PI/2}" xyz="-0.1 0.5 -0.1" />
@@ -52,6 +106,13 @@
             </geometry>
         </visual>
+        <collision>
+            <origin rpy="0 0 -${PI/2}" xyz="-0.1 0.5 -0.1" />
+            <geometry>
+                <mesh filename="package://arduino_bot_description/mesh/right_finger.STL" scale="0.01 0.01 0.01" />
+            </geometry>
+        </collision>
     </link>
     <link name="gripper_left">
+        <xacro:default_inertial mass="0.01" />
         <visual>
             <origin rpy="0 0 -${PI/2}" xyz="-0.04 0.5 -0.1" />
@@ -60,4 +121,10 @@
             </geometry>
         </visual>
+        <collision>
+            <origin rpy="0 0 -${PI/2}" xyz="-0.04 0.5 -0.1" />
+            <geometry>
+                <mesh filename="package://arduino_bot_description/mesh/left_finger.STL" scale="0.01 0.01 0.01" />
+            </geometry>
+        </collision>
     </link>
     <link name="tool_link" />
@@ -108,8 +175,27 @@
         <mimic joint="joint_4" offset="0" multiplier="-1" />
     </joint>
-    <joint name="gripper_right" type="fixed">
+    <joint name="gripper_right_to_tool" type="fixed">
         <parent link="gripper_right"/>
         <child link="tool_link"/>
         <origin rpy="0 0 0" xyz="0 0 0" />
     </joint>
+    <xacro:default_transmission number="1" />
+    <xacro:default_transmission number="2" />
+    <xacro:default_transmission number="3" />
+    <xacro:default_transmission number="4" />
+    <gazebo>
+        <plugin name="gazebo_ros_control" filename="libgazebo_ros_control.so">
+            <robotNamespace>/arduino_bot</robotNamespace>
+            <robotSimType>gazebo_ros_control/DefaultRobotHWSim</robotSimType>
+            <legacyModeNS>true</legacyModeNS>
+        </plugin>
+        <plugin name="joint_5_mimic_4" filename="libroboticsgroup_gazebo_mimic_joint_plugin.so">
+            <joint>joint_4</joint>
+            <mimicJoint>joint_5</mimicJoint>
+            <multiplier>-1.0</multiplier>
+            <offset>0</offset>
+            <maxEffort>${effort}</maxEffort>
+            <robotNamespace>/arduino_bot</robotNamespace>
+        </plugin>
+    </gazebo>
 </robot>
